Commit message: moved base_link between the rear wheels

File: simulation/ackermann_vehicle/ackermann_vehicle_description/urdf/em_3905.urdf.xacro (robot description, xacro)
@@ -347,4 +347,7 @@
     <parent link="base_link"/>
     <child link="chassis"/>
+    <origin xyz="	${wheelbase / 2}
+					0
+					0"/>
   </joint>
   <!-- Batteries -->
